File: data.kicad_sch (KiCad schematic)
At the start: 26 parts, among them J2 USB_C_Receptacle, U11 FT601Q, U12 HD3SS3220, U13 ABM8-30.000MHZ-D1X-T

Commit message: some more fpga work
Connections:
- net FT_CLK: now reaches U11.58 (CLK)
Changed lines of the file:
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@@
+		)
+	)
+	(global_label "FT_CLK"
+		(shape input)
+		(at 186.69 31.75 0)
+		(fields_autoplaced yes)
+		(effects
+			(font
+				(size 1.27 1.27)
+			)
+			(justify left)
+		)
+		(property "Intersheetrefs" "${INTERSHEET_REFS}"
+			(at 196.2671 31.75 0)
+			(effects
+				(font
+					(size 1.27 1.27)
+				)
+				(justify left)
+				(hide yes)
+			)
 		)
 	)

Commit message: i dont even remember what i did
Parts:
- removed C68, C69: 100n, Capacitor_SMD:C_0402_1005Metric, symbol Device:C
- added C26, C28, C31: 100n, Capacitor_SMD:C_0402_1005Metric, symbol Device:C
- added R41: 10K, Resistor_SMD:R_0402_1005Metric, symbol Device:R_US
- added R42: 22, Resistor_SMD:R_0402_1005Metric, symbol Device:R_US
- J2: value USB_C_Receptacle -> GSB4D313302Y1HR; footprint (none) -> Connector_USB:USB_C_Receptacle_Amphenol_12401610E4-2A
- R33, R34: value 10k -> 10K
- U12: footprint (none) -> hfsdr:HD3SS3220IRNHR
Connections:
- net FT_CLK: now also R42.2; no longer U11.58 (CLK)
- net GND: now also C26.2
- net VCC_3.3V: now also R33.2, R34.2, R41.2; no longer R33.1, R34.1
- net RX2-: now reaches J2.A10 (RX2-), U12.18 (RX2n)
- net RX2+: now reaches J2.A11 (RX2+), U12.19 (RX2p)
- net TX1+: now reaches J2.A2 (TX1+)
- net TX1+: now also C28.1
- net TX1-: now reaches J2.A3 (TX1-)
- net TX1-: now also C31.1
- net RX1-: now reaches J2.B10 (RX1-), U12.14 (RX1n)
- net RX1+: now reaches J2.B11 (RX1+), U12.15 (RX1p)
- net TX2+: now reaches C71.1, J2.B2 (TX2+)
- net TX2-: now reaches C70.1, J2.B3 (TX2-)
- net TX1P: now reaches U12.17 (TX1p)
- net TX1P: now also C31.2
- net TX1N: now reaches U12.16 (TX1n)
- net TX1N: now also C28.2
- net FT_SIWUn: now reaches U11.10 (~{SIWU})
- net FT_SIWUn: now also R33.1; no longer R34.2
- net FT_RESETn: now reaches U11.15 (~{RESET})
- net FT_RESETn: now also R34.1, C26.1; no longer R33.2
- net FT_BE0: now reaches U11.4 (BE_0)
- net FT_D0: now reaches U11.40 (DATA_0)
- net FT_D1: now reaches U11.41 (DATA_1)
- net FT_D2: now reaches U11.42 (DATA_2)
- net FT_D3: now reaches U11.43 (DATA_3)
- net FT_D4: now reaches U11.44 (DATA_4)
- net FT_D5: now reaches U11.45 (DATA_5)
- net FT_D6: now reaches U11.46 (DATA_6)
- net FT_D7: now reaches U11.47 (DATA_7)
- net FT_BE1: now reaches U11.5 (BE_1)
- net FT_D8: now reaches U11.50 (DATA_8)
- net FT_D9: now reaches U11.51 (DATA_9)
- net FT_D10: now reaches U11.52 (DATA_10)
- net FT_D11: now reaches U11.53 (DATA_11)
- net FT_D12: now reaches U11.54 (DATA_12)
- net FT_D13: now reaches U11.55 (DATA_13)
- net FT_D14: now reaches U11.56 (DATA_14)
- net FT_D15: now reaches U11.57 (DATA_15)
- net FT_BE2: now reaches U11.6 (BE_2)
- net FT_D16: now reaches U11.60 (DATA_16)
- net FT_D17: now reaches U11.61 (DATA_17)
- net FT_D18: now reaches U11.62 (DATA_18)
- net FT_D19: now reaches U11.63 (DATA_19)
- net FT_D20: now reaches U11.64 (DATA_20)
- net FT_D21: now reaches U11.65 (DATA_21)
- net FT_D22: now reaches U11.66 (DATA_22)
- net FT_D23: now reaches U11.67 (DATA_23)
- net FT_D24: now reaches U11.69 (DATA_24)
- net FT_BE3: now reaches U11.7 (BE_3)
- net FT_D25: now reaches U11.70 (DATA_25)
- net FT_D26: now reaches U11.71 (DATA_26)
- net FT_D27: now reaches U11.72 (DATA_27)
- net FT_D28: now reaches U11.73 (DATA_28)
- net FT_D29: now reaches U11.74 (DATA_29)
- net FT_D30: now reaches U11.75 (DATA_30)
- net FT_D31: now reaches U11.76 (DATA_31)
- net FT_GPIO0: no longer names the net of U11.17 (GPIO0)
- net FT_GPIO1: no longer names the net of U11.18 (GPIO1)
- net OE_N renamed FT_OEn
- net RD_N renamed FT_RDn
- net RXF_N renamed FT_RXFn
- net TXE_N renamed FT_TXEn
- net USB_WAKEUP renamed FT_WAKEUPn
- net FT_WAKEUPn: now also R41.1
- net WR_N renamed FT_WRn
- new net: R42.1, U11.58 (CLK)
- no-connect marks 3 -> 5
Other:
- note added: "length match!"
- moved on the sheet: C70, C71, J2

Commit message: some moderate pcb work
Parts:
- removed R32, R36: 10k, Resistor_SMD:R_0402_1005Metric, symbol Device:R_US
- added D2, D3: TPD4E05U06DQAR, hfsdr:SON50P135X350X55-14N, symbol hfsdr:TPD4E05U06DQAR
- added R47, R48: 0, Resistor_SMD:R_0402_1005Metric, symbol Device:R_US
- added R49, R50: 0 NC, Resistor_SMD:R_0402_1005Metric, symbol Device:R_US
- added TP1: SBU1, TestPoint:TestPoint_Pad_D1.0mm, symbol Connector:TestPoint
- added TP2: SBU2, TestPoint:TestPoint_Pad_D1.0mm, symbol Connector:TestPoint
- added U4: TPD6E05U06RVZ, Package_SON:Texas_R-PUSON-N14, symbol Power_Protection:TPD6E05U06RVZ
- R31: value 10k -> 4.7k
Connections:
- net D+: now also U4.11 (D2-), U4.4 (NC)
- net D-: now also U4.12 (D2+), U4.3 (NC)
- net GND: now also D2.3 (GND_1), D2.8 (GND_2), D3.3 (GND_1), D3.8 (GND_2), U4.10 (GND), U4.5 (GND); no longer U12.29 (ENn_CC)
- net RX1+: now also D2.5 (D2-), D2.6 (NC_1)
- net RX1-: now also D2.4 (D2+), D2.7 (NC_2)
- net RX2+: now also D3.5 (D2-), D3.6 (NC_1)
- net RX2-: now also D3.4 (D2+), D3.7 (NC_2)
- net TX1+: now also D2.2 (D1-), D2.9 (NC_3)
- net TX1-: now also D2.1 (D1+), D2.10 (NC_4)
- net TX2+: now also D3.2 (D1-), D3.9 (NC_3)
- net TX2-: now also D3.1 (D1+), D3.10 (NC_4)
- net CC1: now reaches U12.2 (CC1)
- net CC1: now also R47.2, R50.2, U4.1 (NC), U4.14 (D1+); no longer J2.A5 (CC1)
- net CSBU1: now reaches J2.A8 (SBU1)
- net CSBU1: now also TP1.1, U4.7 (NC), U4.8 (D3-)
- net CC2: now reaches U12.1 (CC2)
- net CC2: now also R48.2, R49.2, U4.13 (D1-), U4.2 (NC); no longer J2.B5 (CC2)
- net CSBU2: now reaches J2.B8 (SBU2)
- net CSBU2: now also TP2.1, U4.6 (NC), U4.9 (D3+)
- net TX2N: now reaches C70.2, U12.20 (TX2n)
- net TX2P: now reaches C71.2, U12.21 (TX2p)
- net MUX_I2C_ADDR: now reaches U12.22 (ADDR)
- net I2C_INTR renamed MUX_I2C_INTR
- net SCL renamed MUX_SCL
- net SDA renamed MUX_SDA
- net USB_ID renamed MUX_USB_ID
- new net C_CC1: J2.A5 (CC1), R47.1, R49.1
- new net C_CC2: J2.B5 (CC2), R48.1, R50.1
- new net MUX_ENn_CC: U12.29 (ENn_CC)
- no-connect marks 5 -> 3
Other:
- note removed: "I2C addr 0x67"
- note removed: "active low enable mux"
- moved on the sheet: C26, C73, R33, R34, R41
