File: dac.kicad_sch (KiCad schematic)
At the start: 1 part, among them IC2 AD9707BCPZ

Commit message: some moderate pcb work
Parts:
- removed IC2: AD9707BCPZ, Package_CSP:LFCSP-32-1EP_5x5mm_P0.5mm_EP3.1x3.1mm_ThermalVias, symbol hfsdr:AD9707BCPZ
Changed lines of the file:
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@@
 	(generator_version "8.0")
 	(paper "A4")
-	(symbol
-		(lib_id "hfsdr:AD9707BCPZ")
-		(at 80.01 93.98 0)
-		(unit 1)
-		(exclude_from_sim no)
-		(in_bom yes)
-		(on_board yes)
-		(dnp no)
-		(fields_autoplaced yes)
-		(property "Reference" "IC2"
-			(at 123.19 87.6614 0)
-			(effects
-				(font
-					(size 1.27 1.27)
-				)
-			)
-		)
-		(property "Value" "AD9707BCPZ"
-			(at 123.19 90.2014 0)
-			(effects
-				(font
-					(size 1.27 1.27)
-				)
-			)
-		)
-		(property "Footprint" "Package_CSP:LFCSP-32-1EP_5x5mm_P0.5mm_EP3.1x3.1mm_ThermalVias"
-			(at 116.84 173.66 0)
-			(effects
-				(font
-					(size 1.27 1.27)
-				)
-				(justify left top)
-				(hide yes)
-			)
-		)
-		(property "Datasheet" "http://www.analog.com/media/en/technical-documentation/data-sheets/AD9704_9705_9706_9707.pdf"
-			(at 116.84 273.66 0)
-			(effects
-				(font
-					(size 1.27 1.27)
-				)
-				(justify left top)
-				(hide yes)
-			)
-		)
-		(property "Description" "AD9707BCPZ, 14 bit-Bit DAC 175Msps, Parallel, 32-Pin LFCSP EP"
-			(at 80.01 93.98 0)
-			(effects
-				(font
-					(size 1.27 1.27)
-				)
-				(hide yes)
-			)
-		)
-		(property "Height" "1"
-			(at 116.84 473.66 0)
-			(effects
-				(font
-					(size 1.27 1.27)
-				)
-				(justify left top)
-				(hide yes)
-			)
-		)
-		(property "Mouser Part Number" "584-AD9707BCPZ"
-			(at 116.84 573.66 0)
-			(effects
-				(font
-					(size 1.27 1.27)
-				)
-				(justify left top)
-				(hide yes)
-			)
-		)
-		(property "Mouser Price/Stock" "https://www.mouser.co.uk/ProductDetail/Analog-Devices/AD9707BCPZ?qs=BpaRKvA4VqGcqD6UIm7zog%3D%3D"
-			(at 116.84 673.66 0)
-			(effects
-				(font
-					(size 1.27 1.27)
-				)
-				(justify left top)
-				(hide yes)
-			)
-		)
-		(property "Manufacturer_Name" "Analog Devices"
-			(at 116.84 773.66 0)
-			(effects
-				(font
-					(size 1.27 1.27)
-				)
-				(justify left top)
-				(hide yes)
-			)
-		)
-		(property "Manufacturer_Part_Number" "AD9707BCPZ"
-			(at 116.84 873.66 0)
-			(effects
-				(font
-					(size 1.27 1.27)
-				)
-				(justify left top)
-				(hide yes)
-			)
-		)
-		(pin "30"
-		)
-		(pin "9"
-		)
-		(pin "1"
-		)
-		(pin "12"
-		)
-		(pin "33"
-		)
-		(pin "19"
-		)
-		(pin "32"
-		)
-		(pin "17"
-		)
-		(pin "7"
-		)
-		(pin "6"
-		)
-		(pin "22"
-		)
-		(pin "31"
-		)
-		(pin "23"
-		)
-		(pin "8"
-		)
-		(pin "13"
-		)
-		(pin "21"
-		)
-		(pin "4"
-		)
-		(pin "24"
-		)
-		(pin "14"
-		)
-		(pin "29"
-		)
-		(pin "20"
-		)
-		(pin "2"
-		)
-		(pin "16"
-		)
-		(pin "3"
-		)
-		(pin "15"
-		)
-		(pin "26"
-		)
-		(pin "18"
-		)
-		(pin "27"
-		)
-		(pin "11"
-		)
-		(pin "28"
-		)
-		(pin "10"
-		)
-		(pin "5"
-		)
-		(pin "25"
-		)
-		(instances
-			(project ""
-				(path "/b0f4ea81-e287-4b08-8f8c-7fcbaea1e477/009070e2-36b6-44f8-956b-7e8b135b9b63"
-					(reference "IC2")
-					(unit 1)
-				)
-			)
-		)
-	)
 )

Commit message: dac work
Parts:
- added C133, C136: 0.1u, Capacitor_SMD:C_0402_1005Metric, symbol Device:C
- added C134: 10n, Capacitor_SMD:C_0402_1005Metric, symbol Device:C
- added C135: 10u, Capacitor_SMD:C_0402_1005Metric, symbol Device:C
- added C137, C144: 56p, Capacitor_SMD:C_0402_1005Metric, symbol Device:C
- added C138: 12p, Capacitor_SMD:C_0402_1005Metric, symbol Device:C
- added C139, C145: 82p, Capacitor_SMD:C_0402_1005Metric, symbol Device:C
- added C140: 62p, Capacitor_SMD:C_0402_1005Metric, symbol Device:C
- added C141, C146: 75p, Capacitor_SMD:C_0402_1005Metric, symbol Device:C
- added C142: 43p, Capacitor_SMD:C_0402_1005Metric, symbol Device:C
- added C143, C147: 47p, Capacitor_SMD:C_0402_1005Metric, symbol Device:C
- added IC2: AD9707BCPZ, Package_CSP:LFCSP-32-1EP_5x5mm_P0.5mm_EP3.1x3.1mm_ThermalVias, symbol hfsdr:AD9707BCPZ
- added L5: 330n, Inductor_SMD:L_0402_1005Metric, symbol Device:L
- added L6: 240n, Inductor_SMD:L_0402_1005Metric, symbol Device:L
- added L7: 270n, Inductor_SMD:L_0402_1005Metric, symbol Device:L
- added R3: 1k, Resistor_SMD:R_0402_1005Metric, symbol Device:R_US
- added TR1: ADT4-6T, RF_Mini-Circuits:Mini-Circuits_CD637_H5.23mm, symbol Transformer:ADT4-6T
Connections:
- new net: C140.2, C141.1, C142.1, C146.2, L6.2, L7.1
- new net: C142.2, C143.1, C147.2, L7.2
- new net: C137.1, C138.1, C144.2, L5.1
- new net: C134.1, C135.1, C136.1
- new net: C134.2, C135.2, C136.2
- new net: C138.2, C139.1, C140.1, C145.2, L5.2, L6.1
- new net AGND: C133.2, C137.2, C139.2, C141.2, C143.2, C144.1, C145.1, C146.1, C147.1
- new net IOUTA: IC2.21 (IOUTA), R3.2, TR1.6
- new net IOUTB: IC2.20 (IOUTB), R3.1, TR1.4
- new net REFIO: C133.1, IC2.23 (REFIO)
