File: fpga.kicad_sch (KiCad schematic)
At the start: 0 parts

Commit message: some more fpga work
Parts:
- added IC1: LFE5U-25F-6BG256C, hfsdr:BGA256C80P16X16_1400X1400X170, symbol hfsdr:LFE5U-25F-6BG256C
- added J1: JTAG, Connector_PinHeader_1.27mm:PinHeader_2x05_P1.27mm_Vertical, symbol Connector:Conn_ARM_JTAG_SWD_10
- added R38, R40: 4.7k, Resistor_SMD:R_0402_1005Metric, symbol Device:R_US
- added R39: 1.5k, Resistor_SMD:R_0402_1005Metric, symbol Device:R_US
- added U1: W25Q128JVP, Package_SON:WSON-8-1EP_6x5mm_P1.27mm_EP3.4x4.3mm, symbol Memory_Flash:W25Q128JVP
Connections:
- new net FPGA_RESET: IC1.M8 (PB15B), IC1.R9 (PROGRAMN), J1.10 (~{RESET})
- new net GND: IC1.A1 (GND_1), IC1.A16 (GND_2), IC1.D15 (GND_4), IC1.D2 (GND_3), IC1.F8 (GND_5), IC1.F9 (GND_6), IC1.G10 (GND_8), IC1.G8 (GND_7), IC1.H1 (GND_9), IC1.H10 (GND_12), IC1.H16 (GND_13), IC1.H8 (GND_10), IC1.H9 (GND_11), IC1.J10 (GND_16), IC1.J8 (GND_14), IC1.J9 (GND_15), IC1.K10 (GND_21), IC1.K6 (GND_17), IC1.K7 (GND_18), IC1.K8 (GND_19), IC1.K9 (GND_20), IC1.N10 (CFG_0), IC1.N15 (GND_23), IC1.N2 (GND_22), IC1.R10 (CFG_2), IC1.T1 (GND_24), IC1.T12 (GND_26), IC1.T16 (GND_27), IC1.T5 (GND_25), J1.3 (GND), J1.5 (GND), J1.9 (GNDDetect), R38.1, U1.4 (GND)
- new net IO_MISO: IC1.T6 (PB4A)
- new net IO_MOSI: IC1.R6 (PB4B)
- new net IO_SCK: IC1.R8 (PB13A)
- new net JTAG_TCK: IC1.T10 (TCK), J1.4 (SWCLK/TCK), R38.2
- new net JTAG_TDI: IC1.R11 (TDI), J1.8 (NC/TDI)
- new net JTAG_TDO: IC1.M10 (TDO), J1.6 (SWO/TDO)
- new net JTAG_TMS: IC1.T11 (TMS), J1.2 (SWDIO/TMS)
- new net P1.1V: IC1.G6 (VCC_1), IC1.G7 (VCC_2), IC1.G9 (VCC_3), IC1.L10 (VCC_6), IC1.L8 (VCC_4), IC1.L9 (VCC_5)
- new net P2.5V: IC1.G11 (VCCAUX_1), IC1.L7 (VCCAUX_2)
- new net P3.3V: IC1.L6 (VCCIO8), IC1.P10 (CFG_1), J1.1 (VTref), R39.2, R40.2, U1.8 (VCC)
- new net QSPI_D2: IC1.M7 (PB9B), U1.3 (IO2)
- new net QSPI_D3: IC1.N7 (PB9A), U1.7 (IO3)
- new net SPICFG_MISO: IC1.T7 (PB11A), U1.2 (DO(IO1))
- new net SPICFG_MOSI: IC1.T8 (PB11B), U1.5 (DI(IO0))
- new net SPICFG_SCK: IC1.N9 (CCLK/MCLK/SCK), R39.1, U1.6 (CLK)
- new net SPICFG_SS: IC1.N8 (PB15A), R40.1, U1.1 (~{CS})
- no-connect marks 0 -> 2

Commit message: i dont even remember what i did
Parts:
- added C100, C102, C104, C106, C108, C110, C112, C114, C116, C27, C36, C41, C82, C92, C93, C94, C96, C98: 0.1u, Capacitor_SMD:C_0402_1005Metric, symbol Device:C
- added C101, C103, C105, C107, C109, C111, C113, C115, C32, C33, C35, C37, C38, C39, C42, C68, C69, C83, C84, C85, C86, C87, C88, C89, C90, C91, C95, C97, C99: 10u, Capacitor_SMD:C_0402_1005Metric, symbol Device:C
- added R43, R44, R45: 4.7k, Resistor_SMD:R_0402_1005Metric, symbol Device:R_US
- added R46: 120, Resistor_SMD:R_0402_1005Metric, symbol Device:R_US
Connections:
- net GND: now also C100.2, C101.2, C102.2, C103.2, C104.2, C105.2, C106.2, C107.2, C108.2, C109.2, C110.2, C111.2, C112.2, C113.2, C114.2, C115.2, C116.2, C27.2, C32.2, C33.2, C35.2, C36.2, C37.2, C38.2, C39.2, C41.2, C42.2, C68.2, C69.2, C82.2, C83.2, C84.2, C85.2, C86.2, C87.2, C88.2, C89.2, C90.2, C91.2, C92.2, C93.2, C94.2, C99.2
- net JTAG_TDI: now also R45.1
- net JTAG_TDO: now also R44.1
- net JTAG_TMS: now also R43.1
- net P1.1V: now also C32.1, C33.1, C35.1, C36.1, C37.1, C38.1, C39.1, C41.1, C42.1, C68.1, C69.1, C82.1, C83.1, C84.1, C85.1, C86.1, C87.1, C88.1, C89.1, C90.1, C91.1, C92.1, C93.1, C94.1
- net P2.5V: now also R46.1; no longer IC1.G11 (VCCAUX_1), IC1.L7 (VCCAUX_2)
- net P3.3V: now also IC1.H6 (VCCIO7_1), IC1.H7 (VCCIO7_2), IC1.J6 (VCCIO6_1), IC1.J7 (VCCIO6_2), C107.1, C108.1, C109.1, C110.1, C111.1, C112.1, C113.1, C114.1, C115.1, C116.1, C27.1, R43.2, R44.2, R45.2
- net D1: now reaches IC1.B15 (PR2B)
- net D0: now reaches IC1.B16 (PR2A)
- net D2: now reaches IC1.C14 (PR2C)
- net D5: now reaches IC1.C15 (PR5B)
- net D4: now reaches IC1.C16 (PR5A)
- net D3: now reaches IC1.D14 (PR2D)
- net D8: now reaches IC1.D16 (PR8A)
- net D6: now reaches IC1.E14 (PR5C)
- net D9: now reaches IC1.E15 (PR8B)
- net D10: now reaches IC1.E16 (PR11D)
- net D7: now reaches IC1.F14 (PR5D)
- net DCO: now reaches IC1.F15 (PR11C)
- net D11: now reaches IC1.F16 (PR14A)
- net D12: now reaches IC1.G15 (PR14B)
- net D13: now reaches IC1.G16 (PR20A)
- net DRVDD: now reaches IC1.H11 (VCCIO2_1)
- net DRVDD: now also IC1.J11 (VCCIO2_2), IC1.K11 (VCCIO3_1), IC1.L11 (VCCIO3_2), C100.1, C101.1, C102.1, C103.1, C104.1, C105.1, C106.1, C99.1
- net FT_D31: now reaches IC1.C2 (PL5B)
- net FT_D30: now reaches IC1.C3 (PL2C)
- net FT_D29: now reaches IC1.D1 (PL8A)
- net FT_D28: now reaches IC1.D3 (PL2D)
- net FT_D27: now reaches IC1.E1 (PL11D)
- net FT_D26: now reaches IC1.E2 (PL8B)
- net FT_D25: now reaches IC1.E3 (PL5C)
- net FT_D24: now reaches IC1.F1 (PL14A)
- net FT_D23: now reaches IC1.F2 (PL11C)
- net FT_D22: now reaches IC1.F3 (PL5D)
- net FT_D21: now reaches IC1.G1 (PL20A)
- net FT_D20: now reaches IC1.G2 (PL14B)
- net FT_D19: now reaches IC1.G3 (PL14C)
- net FT_D18: now reaches IC1.H2 (PL20B)
- net FT_D17: now reaches IC1.H3 (PL14D)
- net FT_D16: now reaches IC1.J1 (PL23A)
- net FT_D15: now reaches IC1.J2 (PL23B)
- net FT_D14: now reaches IC1.J3 (PL20C)
- net FT_D13: now reaches IC1.K1 (PL23C)
- net FT_D12: now reaches IC1.K2 (PL23D)
- net FT_D11: now reaches IC1.K3 (PL20D)
- net FT_D10: now reaches IC1.L1 (PL26A)
- net FT_D9: now reaches IC1.L2 (PL26B)
- net FT_D8: now reaches IC1.L3 (PL32C)
- net FT_D7: now reaches IC1.M1 (PL26C)
- net FT_D6: now reaches IC1.M2 (PL26D)
- net FT_D5: now reaches IC1.M3 (PL32D)
- net FT_D3: now reaches IC1.N1 (PL32A)
- net FT_D4: now reaches IC1.N3 (PL35D)
- net FT_BE3: now reaches IC1.P1 (PL35A)
- net FT_D2: now reaches IC1.P2 (PL32B)
- net FT_BE2: now reaches IC1.R1 (PL35B)
- net FT_D1: now reaches IC1.R2 (PL38C)
- net FT_D0: now reaches IC1.R3 (PL41B)
- net FT_BE0: now reaches IC1.T2 (PL38D)
- net FT_BE1: now reaches IC1.T3 (PL41D)
- new net: C95.1, C96.1, C97.1, C98.1, IC1.G11 (VCCAUX_1), IC1.L7 (VCCAUX_2), R46.2
- new net: C95.2, C96.2, C97.2, C98.2
- no-connect marks 2 -> 6
Other:
- note added: "1.8v io"
- note added: "3.3v io"
- note added: "bank 2+3"
- note added: "bank 6+7"
- note added: "bank 8"
- note added: "core"
- moved on the sheet: IC1B, IC1C, IC1D, IC1F, R38, R39

Commit message: some moderate pcb work
Parts:
- added C118, C120, C122, C124: 10u, Capacitor_SMD:C_0402_1005Metric, symbol Device:C
- added C119, C121, C123, C125: 0.1u, Capacitor_SMD:C_0402_1005Metric, symbol Device:C
Connections:
- net ADC_CSB: now also IC1.K15 (PR23D)
- net ADC_MODE/OR: now also IC1.J16 (PR23A)
- net ADC_SCLK: now also IC1.K16 (PR23C)
- net ADC_SDIO: now also IC1.J15 (PR23B)
- net GND: now also C118.2, C119.2, C120.2, C121.2, C122.2, C123.2, C124.2, C125.2
- net P3.3V: now also IC1.F10 (VCCIO1_1), IC1.F11 (VCCIO1_2), IC1.F6 (VCCIO0_1), IC1.F7 (VCCIO0_2), C118.1, C119.1, C120.1, C121.1, C122.1, C123.1, C124.1, C125.1
- net VGA_CSB: now also IC1.A2 (PT4A)
- net VGA_ENABLE: now also IC1.A4 (PT6B)
- net VGA_SCLK: now also IC1.B3 (PT4B)
- net VGA_SDIO: now also IC1.A3 (PT6A)
- net PORT_DIR: now reaches IC1.A5 (PT18A)
- net MUX_SDA: now reaches IC1.B4 (PT11B)
- net EN_MUX: now reaches IC1.B5 (PT15B)
- net MUX_SCL: now reaches IC1.C4 (PT11A)
- net MUX_I2C_ADDR: now reaches IC1.C5 (PT15A)
- net MUX_USB_ID: now reaches IC1.D4 (PT9B)
- net MUX_I2C_INTR: now reaches IC1.D5 (PT13B)
- net MUX_ENn_CC: now reaches IC1.E4 (PT9A)
- net VCONN_FAULT: now reaches IC1.E5 (PT13A)
- no-connect marks 6 -> 7
Other:
- note added: "bank 0+1"
- moved on the sheet: C107, C108, C109, C110, C111, C112, C113, C114, C115, C116, IC1C, IC1D

Commit message: dac work
Connections:
- net ADC_CSB: no longer IC1.K15 (PR23D)
- net ADC_MODE/OR: no longer IC1.J16 (PR23A)
- net ADC_SCLK: no longer IC1.K16 (PR23C)
- net ADC_SDIO: no longer IC1.J15 (PR23B)
- net D10: now also IC1.M13 (PR35C); no longer IC1.E16 (PR11D)
- net D11: now also IC1.N14 (PR35D); no longer IC1.F16 (PR14A)
- net D12: now also IC1.P15 (PR32B); no longer IC1.G15 (PR14B)
- net D13: now also IC1.R15 (PR38C); no longer IC1.G16 (PR20A)
- net D4: now also IC1.F13 (PR8C); no longer IC1.C16 (PR5A)
- net D5: now also IC1.G13 (PR11B); no longer IC1.C15 (PR5B)
- net D6: now also IC1.H13 (PR17B); no longer IC1.E14 (PR5C)
- net D7: now also IC1.J13 (PR17C); no longer IC1.F14 (PR5D)
- net D8: now also IC1.K13 (PR29A); no longer IC1.D16 (PR8A)
- net D9: now also IC1.L13 (PR29C); no longer IC1.E15 (PR8B)
- net DCO: now also IC1.R16 (PR35B); no longer IC1.F15 (PR11C)
