File: hfsdr.kicad_pcb (KiCad board)
At the start: 4 copper layers, 140 x 65 mm, 201 parts, among them IC1 LFE5U-25F-6BG256C, J1 JTAG, J2 GSB4D313302Y1HR, U1 W25Q128JVP, U10 ADA4938-1, U11 FT601Q, U12 HD3SS3220, U13 ABM8-30.000MHZ-D1X-T, U14 AD9649, U4 TPD6E05U06RVZ, U5 TLV77333PDBVR, U6 AD9515, U7 ADL5206, U8 AP2205-50Y-13, U9 AP2205-50Y-13, Y1 590BD80M0000DG

Commit message: dac work
Parts:
- moved U11 16.6 mm to (119.4, 146.9), turned to -90 degrees
- moved R29 15.6 mm to (105.5, 151.1)
- moved C77 15.6 mm to (94.5, 152.1)
- moved C78 15.6 mm to (96.5, 149.1)
- moved U13 15.6 mm to (99.9, 152.3)
- moved U8 11.1 mm to (175.5, 98.9)
- moved IC1 5.75 mm to (139.3, 147.0)
- moved R4 3.11 mm to (100.7, 104.7)
- moved RF1 1.36 mm to (198.0, 144.8)
- moved C21 1.10 mm to (99.2, 105.2)
- moved J2 0.95 mm to (65.2, 150.5)
Connections:
- IC1 pad C15: D5 -> unconnected-(IC1C-PR5B-PadC15)
- IC1 pad C16: D4 -> unconnected-(IC1C-PR5A-PadC16)
- IC1 pad D16: D8 -> unconnected-(IC1C-PR8A-PadD16)
- IC1 pad E14: D6 -> unconnected-(IC1C-PR5C-PadE14)
- IC1 pad E15: D9 -> unconnected-(IC1C-PR8B-PadE15)
- IC1 pad E16: D10 -> unconnected-(IC1C-PR11D-PadE16)
- IC1 pad F13: unconnected-(IC1C-PR8C-PadF13) -> D4
- IC1 pad F14: D7 -> unconnected-(IC1C-PR5D-PadF14)
- IC1 pad F15: DCO -> unconnected-(IC1C-PR11C-PadF15)
- IC1 pad F16: D11 -> unconnected-(IC1C-PR14A-PadF16)
- IC1 pad G13: unconnected-(IC1C-PR11B-PadG13) -> D5
- IC1 pad G15: D12 -> unconnected-(IC1C-PR14B-PadG15)
- IC1 pad G16: D13 -> unconnected-(IC1C-PR20A-PadG16)
- IC1 pad H13: unconnected-(IC1C-PR17B-PadH13) -> D6
- IC1 pad J13: unconnected-(IC1C-PR17C-PadJ13) -> D7
- IC1 pad J15: ADC_SDIO -> unconnected-(IC1C-PR23B-PadJ15)
- IC1 pad J16: ADC_MODE/OR -> unconnected-(IC1C-PR23A-PadJ16)
- IC1 pad K13: unconnected-(IC1C-PR29A-PadK13) -> D8
- IC1 pad K15: ADC_CSB -> unconnected-(IC1C-PR23D-PadK15)
- IC1 pad K16: ADC_SCLK -> unconnected-(IC1C-PR23C-PadK16)
- IC1 pad L13: unconnected-(IC1C-PR29C-PadL13) -> D9
- IC1 pad M13: unconnected-(IC1C-PR35C-PadM13) -> D10
- IC1 pad N14: unconnected-(IC1C-PR35D-PadN14) -> D11
- IC1 pad P15: unconnected-(IC1C-PR32B-PadP15) -> D12
- IC1 pad R15: unconnected-(IC1C-PR38C-PadR15) -> D13
- IC1 pad R16: unconnected-(IC1C-PR35B-PadR16) -> DCO
Routing:
- net AGND: track 67.7 -> 52.8 mm, vias 74 -> 67
- net D2: track 2.77 -> 10.8 mm
- net D8: track 2.90 -> 10.8 mm
- net D3: track 3.17 -> 10.7 mm
- net D4: track 3.22 -> 10.7 mm
- net D1: track 3.51 -> 10.8 mm
- net D5: track 3.55 -> 10.8 mm
- net D9: track 3.68 -> 10.8 mm
- net D0: track 4.15 -> 10.8 mm
- net Net-(D1-A2): track 6.34 -> 0.00 mm
- net D7: track 4.47 -> 10.8 mm
- net D6: track 4.65 -> 10.8 mm
- net D10: track 4.82 -> 10.8 mm
- net D11: track 5.78 -> 10.8 mm
- net Net-(C22-Pad1): track 0.00 -> 4.24 mm
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